Commit message: rails extended, new model added
gripper speed extended

File: Phase_2_codebase/rsc/rail1.urdf (robot description, URDF)
Before this commit: robot rail1, 3 links, 2 joints
Links:
- link Untitled.066: geometry collision box size=6.0 0.35 0.01; visual box size=6.0 0.35 0.01
- link Untitled.067: geometry collision box size=6.0 0.01 0.05; visual box size=6.0 0.01 0.05
- link Untitled.068: geometry collision box size=6.0 0.01 0.05; visual box size=6.0 0.01 0.05

Commit message: constraints added to rails

File: Phase_2_codebase/rsc/rail1.urdf (robot description, URDF)
Before this commit: robot rail1, 3 links, 2 joints
Links:
- link Untitled.066: geometry collision box size=5.0 0.35 0.01; visual box size=5.0 0.35 0.01
- link Untitled.067: geometry collision box size=5.0 0.01 0.05; visual box size=5.0 0.01 0.05
- link Untitled.068: geometry collision box size=5.0 0.01 0.05; visual box size=5.0 0.01 0.05
