Commit message: suction added,
decision making to be fine tuned

File: Phase_2_codebase/rsc/bot_acha.urdf (robot description, URDF)
Before this commit: robot bot, 64 links, 63 joints
Links:
- added link Untitled.039, mass 0.01; collision box size=0.08 0.005 0.06; visual box size=0.08 0.005 0.06
- added link Untitled.040, mass 0.05; collision box size=0.08 0.005 0.08; visual box size=0.08 0.005 0.08
- link Untitled.036: geometry collision box size=0.08 0.145 0.04; visual box size=0.08 0.15 0.08
- link Untitled.037: mass 0.05 -> 0.01; geometry collision box size=0.08 0.005 0.06; visual box size=0.08 0.005 0.06
- link Untitled.038: geometry collision box size=0.08 0.005 0.08; visual box size=0.08 0.005 0.08
- link Untitled.047: geometry collision box size=0.04 0.03 0.01; visual box size=0.04 0.03 0.01
- link Untitled.050: mass 4.0 -> 3.0
- link Untitled.051: mass 4.0 -> 3.0
Joints:
- added joint Untitled.039: type fixed, parent Untitled.040, child Untitled.039, origin xyz=0 0.05 0 rpy=1.13446 0 0
- added joint Untitled.040: type prismatic, parent Untitled.036, child Untitled.040, origin xyz=0 0.075 -0.08044 rpy=-1.5708 0 0, axis 0 0 1.0, limit lower=-1.2931 upper=1.29 effort=0.1 velocity=1.0
- joint Untitled.018: origin xyz=0 0.04 -0.04 rpy=0 0 0 -> xyz=0 0.02 -0.04 rpy=0 0 0
- joint Untitled.037: origin xyz=0 -0.0625 -0.09126 rpy=1.5708 0 0 -> xyz=0 -0.05 0 rpy=-1.13446 0 0; parent Untitled.036 -> Untitled.038
- joint Untitled.038: axis 0 0 1.0 -> (none); limit lower=-1.6 upper=1.6 effort=0.1 velocity=0.05 -> (none); origin xyz=0 0.0825 -0.09126 rpy=1.5708 0 0 -> xyz=0 -0.075 -0.08044 rpy=1.5708 0 0; type prismatic -> fixed
- joint Untitled.041: origin xyz=0.04032 -0.00214 -0.00337 rpy=0 0 0 -> xyz=0.07032 -0.00214 -0.00337 rpy=0 0 0
