Commit message: new bot added

File: Phase_2_codebase/rsc/bot.urdf (robot description, URDF)
Before this commit: robot bot, 64 links, 63 joints
Links:
- added link Untitled.039, mass 0.001; visual mesh filename=L bracket.stl scale=0.00186 0.00228 0.00167
- added link Untitled.040, mass 0.001; visual mesh filename=L bracket.stl scale=0.00232 0.00228 0.00167
- added link Untitled.073, mass 0.001; visual mesh filename=L bracket.stl scale=0.00186 0.00228 0.00167
- added link Untitled.074, mass 0.001; visual mesh filename=L bracket.stl scale=0.00232 0.00228 0.00167
- added link Untitled.075, mass 0.001; visual mesh filename=L bracket.stl scale=0.00186 0.00228 0.00167
- added link Untitled.076, mass 0.001; visual mesh filename=L bracket.stl scale=0.00232 0.00228 0.00167
- added link Untitled.077, mass 0.001; visual mesh filename=L bracket.stl scale=0.00186 0.00228 0.00167
- added link Untitled.078, mass 0.001; visual mesh filename=L bracket.stl scale=0.00232 0.00228 0.00167
- added link Untitled.079, mass 0.001; visual mesh filename=Original.stl scale=0.1462 0.01681 0.00592
- added link Untitled.080, mass 0.001; visual box size=0.01 0.026 0.05
- added link Untitled.081, mass 0.001; visual box size=0.01 0.026 0.05
- added link Untitled.082, mass 0.001; visual cylinder length=0.06 radius=0.015
- added link Untitled.083, mass 0.001; visual cylinder length=0.06 radius=0.015
- added link Untitled.084, mass 0.001; visual cylinder length=0.06 radius=0.015
- added link Untitled.085, mass 0.001; visual mesh filename=DC Motor.stl scale=0.00227 0.00227 0.00133
- added link Untitled.086, mass 0.001; visual mesh filename=DC Motor.stl scale=0.00227 0.00227 0.00133
- added link Untitled.087, mass 0.001; visual mesh filename=DC Motor.stl scale=0.00227 0.00227 0.00133
- added link Untitled.088, mass 0.001; visual mesh filename=DC Motor.stl scale=0.00227 0.00227 0.00133
- added link Untitled.089, mass 0.001; visual mesh filename=DC Motor.stl scale=0.00227 0.00227 0.00133
- added link Untitled.090, mass 0.001; visual mesh filename=DC Motor.stl scale=0.00227 0.00227 0.00133
- added link Untitled.091, mass 0.001; visual mesh filename=DC Motor.stl scale=0.00227 0.00227 0.00133
- added link Untitled.092, mass 0.001; visual mesh filename=DC Motor.stl scale=0.00227 0.00227 0.00133
- added link Untitled.093, mass 0.001; visual mesh filename=NEMA 17.001.stl scale=0.00099 0.00099 0.00059
- added link Untitled.094, mass 0.001; visual mesh filename=NEMA 17.002.stl scale=0.00099 0.00099 0.00059
- added link Untitled.095, mass 0.001; visual mesh filename=16gear.stl scale=0.00053 0.00053 0.001
- added link Untitled.096, mass 0.001; visual mesh filename=rack.stl scale=0.00089 0.00136 0.004
- link Untitled.004: geometry collision box size=0.4 0.2 0.1; visual box size=0.5 0.2 0.1
- link Untitled.005: geometry collision cylinder length=0.05 radius=0.09; visual mesh filename=Cylinder.004.stl scale=1.0 1.0 1.0
- link Untitled.009: geometry collision box size=0.4 0.2 0.1; visual box size=0.5 0.2 0.1
- link Untitled.036: geometry collision box size=0.04 0.15 0.08; visual box size=0.06 0.15 0.08
- link Untitled.037: geometry collision box size=0.04 0.005 0.1; visual box size=0.06 0.005 0.1
- link Untitled.038: geometry collision box size=0.04 0.005 0.1; visual box size=0.06 0.005 0.1
- link Untitled.045: geometry 
- link Untitled.046: geometry 
- link Untitled.058: geometry visual mesh filename=Original.stl scale=0.1462 0.01681 0.00592
Joints:
- added joint Untitled.039: type fixed, parent Untitled.009, child Untitled.039, origin xyz=-0.025 0.03 0.0476 rpy=1.5708 0 1.5708
- added joint Untitled.040: type fixed, parent Untitled.009, child Untitled.040, origin xyz=-0.025 -0.02 0.0476 rpy=1.5708 0 -3.14159
- added joint Untitled.073: type fixed, parent Untitled.009, child Untitled.073, origin xyz=0.025 -0.02 0.0476 rpy=1.5708 0 -1.5708
- added joint Untitled.074: type fixed, parent Untitled.009, child Untitled.074, origin xyz=0.03 0.03 0.0476 rpy=1.5708 0 0
- added joint Untitled.075: type fixed, parent Untitled.004, child Untitled.075, origin xyz=-0.025 0.025 0.06 rpy=1.5708 0 1.5708
- added joint Untitled.076: type fixed, parent Untitled.004, child Untitled.076, origin xyz=-0.025 -0.025 0.06 rpy=1.5708 0 -3.14159
- added joint Untitled.077: type fixed, parent Untitled.004, child Untitled.077, origin xyz=0.025 -0.025 0.06 rpy=1.5708 0 -1.5708
- added joint Untitled.078: type fixed, parent Untitled.004, child Untitled.078, origin xyz=0.03 0.025 0.06 rpy=1.5708 0 0
- added joint Untitled.079: type fixed, parent Untitled.048, child Untitled.079, origin xyz=-0.11388 1.2511 0.10827 rpy=1.5708 0 1.5708
- added joint Untitled.080: type fixed, parent Untitled.029, child Untitled.080, origin xyz=0.025 0 0.03113 rpy=0 0 0
- added joint Untitled.081: type fixed, parent Untitled.032, child Untitled.081, origin xyz=0.02762 -0.0014 0.03161 rpy=0 0 0
- added joint Untitled.082: type fixed, parent Untitled.027, child Untitled.082, origin xyz=0 -0.035 0.11744 rpy=0 0 0
- added joint Untitled.083: type fixed, parent Untitled.030, child Untitled.083, origin xyz=0 -0.035 0.12198 rpy=0 0 0
- added joint Untitled.084: type fixed, parent Untitled.033, child Untitled.084, origin xyz=0 -0.035 0.11828 rpy=0 0 0
- added joint Untitled.085: type fixed, parent Untitled.003, child Untitled.085, origin xyz=0.05 0 -0.04 rpy=0 0 3.14159
- added joint Untitled.086: type fixed, parent Untitled.002, child Untitled.086, origin xyz=0.03 0 -0.04 rpy=0 0 0
- added joint Untitled.087: type fixed, parent Untitled, child Untitled.087, origin xyz=-0.05 0 -0.04 rpy=0 0 0
- added joint Untitled.088: type fixed, parent Untitled.001, child Untitled.088, origin xyz=-0.03 0 -0.04 rpy=0 0 3.14159
- added joint Untitled.089: type fixed, parent Untitled.016, child Untitled.089, origin xyz=0.04 0.0124 -0.035 rpy=0 0 3.14159
- added joint Untitled.090: type fixed, parent Untitled.014, child Untitled.090, origin xyz=0.02 -0.0124 -0.045 rpy=0 0 0
- added joint Untitled.091: type fixed, parent Untitled.012, child Untitled.091, origin xyz=-0.05 -0.0124 -0.045 rpy=0 0 0
- added joint Untitled.092: type fixed, parent Untitled.010, child Untitled.092, origin xyz=-0.03 0.0124 -0.035 rpy=0 0 3.14159
- added joint Untitled.093: type fixed, parent Untitled.036, child Untitled.093, origin xyz=0.01 -0.01 0.00115 rpy=0 0 0
- added joint Untitled.094: type fixed, parent Untitled.036, child Untitled.094, origin xyz=-0.03 -0.04997 -0.03088 rpy=0 1.5708 0
- added joint Untitled.095: type fixed, parent Untitled.094, child Untitled.095, origin xyz=-0.02003 -0.0025 0.03571 rpy=0 0 0
- added joint Untitled.096: type fixed, parent Untitled.038, child Untitled.096, origin xyz=0 0.05168 0.0085 rpy=0 1.5708 0
- joint Untitled.005: origin xyz=0 0 -0.07 rpy=3.14159 0 0 -> xyz=0.04 0 -0.07 rpy=3.14159 0 0
- joint Untitled.006: origin xyz=0 0 -0.07 rpy=3.14159 0 0 -> xyz=-0.04 0 -0.07 rpy=3.14159 0 0
- joint Untitled.007: origin xyz=0 0 -0.07 rpy=-3.14159 0 0 -> xyz=-0.04 0 -0.07 rpy=-3.14159 0 0
- joint Untitled.008: origin xyz=0 0 -0.07 rpy=-3.14159 0 0 -> xyz=0.04 0 -0.07 rpy=-3.14159 0 0
- joint Untitled.011: origin xyz=0 0 -0.07 rpy=-3.14159 0 0 -> xyz=-0.04 0 -0.07 rpy=-3.14159 0 0
- joint Untitled.013: origin xyz=0 0 -0.07 rpy=3.14159 0 0 -> xyz=-0.04 0 -0.07 rpy=3.14159 0 0
- joint Untitled.015: origin xyz=0 0 -0.07 rpy=3.14159 0 0 -> xyz=0.04 0 -0.07 rpy=3.14159 0 0
- joint Untitled.017: origin xyz=0 0 -0.07 rpy=-3.14159 0 0 -> xyz=0.04 0 -0.07 rpy=-3.14159 0 0

Commit message: new bot

File: Phase_2_codebase/rsc/bot.urdf (robot description, URDF)
Before this commit: robot bot, 90 links, 89 joints
Links:
- added link Untitled.097, mass 0.001; visual mesh filename=Cylinder.003.stl scale=0.77778 0.77778 1.0
- added link Untitled.098, mass 0.001; visual mesh filename=Cylinder.003.stl scale=0.77778 0.77778 1.0
- added link Untitled.099, mass 0.001; visual mesh filename=Cylinder.003.stl scale=0.77778 0.77778 1.0
- added link Untitled.100, mass 0.001; visual mesh filename=Cylinder.003.stl scale=0.77778 0.77778 1.0
- added link Untitled.101, mass 0.001; visual mesh filename=motoreducteur.stl scale=0.00114 0.00446 0.00157
- added link Untitled.102, mass 0.001; visual cylinder length=0.23 radius=0.005
- added link Untitled.104, mass 0.001; visual mesh filename=motoreducteur.stl scale=0.00114 0.00446 0.00157
- added link Untitled.105, mass 0.001; visual cylinder length=0.23 radius=0.005
- added link Untitled.106, mass 0.001; visual mesh filename=L bracket.stl scale=0.00116 0.0016 0.00167
- added link Untitled.107, mass 0.001; visual mesh filename=L bracket.stl scale=0.00116 0.0016 0.00167
- added link Untitled.108, mass 0.001; visual mesh filename=L bracket.stl scale=0.00116 0.0016 0.00167
- added link Untitled.109, mass 0.001; visual mesh filename=L bracket.stl scale=0.00116 0.0016 0.00167
- added link Untitled.110, mass 0.2; collision box size=0.23 0.1 0.06; collision mesh filename=vertical rod.007.stl scale=1.0 1.0 1.0
- added link Untitled.111, mass 0.2; collision box size=0.23 0.1 0.05; collision mesh filename=vertical rod.005.stl scale=1.0 1.0 1.0
- link Untitled.004: geometry collision box size=0.5 0.2 0.1; visual box size=0.5 0.2 0.1
- link Untitled.005: geometry collision cylinder length=0.05 radius=0.07; visual mesh filename=Cylinder.004.stl scale=0.77778 0.77778 1.0
- link Untitled.006: geometry collision cylinder length=0.05 radius=0.07; visual cylinder length=0.05 radius=0.07
- link Untitled.007: geometry collision cylinder length=0.05 radius=0.07; visual cylinder length=0.05 radius=0.07
- link Untitled.008: geometry collision cylinder length=0.05 radius=0.07; visual cylinder length=0.05 radius=0.07
- link Untitled.009: geometry collision box size=0.5 0.2 0.1; visual box size=0.5 0.2 0.1
- link Untitled.011: geometry collision cylinder length=0.05 radius=0.07; visual cylinder length=0.05 radius=0.07
- link Untitled.013: mass 0.25 -> 0.001; geometry visual mesh filename=Pulley T-Mxl-Xl-Htd-Gt2 N-Tooth 20141225-11880-1Y2Kfq6-0.stl scale=0.00021 0.00037 0.005
- link Untitled.015: geometry collision cylinder length=0.05 radius=0.07; visual cylinder length=0.05 radius=0.07
- link Untitled.017: geometry collision cylinder length=0.05 radius=0.07; visual cylinder length=0.05 radius=0.07
- link Untitled.039: geometry visual mesh filename=L bracket.stl scale=0.00116 0.0016 0.00167
- link Untitled.040: geometry visual mesh filename=L bracket.stl scale=0.00116 0.0016 0.00167
- link Untitled.045: mass 1.0 -> 0.001; geometry visual mesh filename=L bracket.stl scale=0.00116 0.0016 0.00167
- link Untitled.046: mass 1.0 -> 0.001; geometry visual mesh filename=L bracket.stl scale=0.00116 0.0016 0.00167
- link Untitled.048: geometry visual box size=0.1 0.07 0.03
- link Untitled.050: mass 4.0 -> 0.001; geometry visual mesh filename=L bracket.stl scale=0.00116 0.0016 0.00167
- link Untitled.051: mass 4.0 -> 0.001; geometry visual mesh filename=L bracket.stl scale=0.00116 0.0016 0.00167
- link Untitled.052: geometry collision mesh filename=horizantal rod.001.stl scale=1.0 1.0 1.0; visual mesh filename=horizantal rod.stl scale=1.02128 1.00001 1.0
- link Untitled.054: mass 0.001 -> 0.25; geometry collision cylinder length=0.05 radius=0.07; visual cylinder length=0.05 radius=0.07
- link Untitled.073: geometry visual mesh filename=L bracket.stl scale=0.00116 0.0016 0.00167
- link Untitled.074: geometry visual mesh filename=L bracket.stl scale=0.00116 0.0016 0.00167
- link Untitled.075: geometry visual mesh filename=L bracket.stl scale=0.00116 0.0016 0.00167
- link Untitled.076: geometry visual mesh filename=L bracket.stl scale=0.00116 0.0016 0.00167
- link Untitled.077: geometry visual mesh filename=L bracket.stl scale=0.00116 0.0016 0.00167
- link Untitled.078: geometry visual mesh filename=L bracket.stl scale=0.00116 0.0016 0.00167
Joints:
- added joint Untitled.097: type continuous, parent Untitled.004, child Untitled.097, origin xyz=-0.00259 0.125 0.0024 rpy=1.5708 0 -3.14159, axis 0 0 1.0, limit effort=0.01 velocity=0.1
- added joint Untitled.098: type continuous, parent Untitled.004, child Untitled.098, origin xyz=-0.00259 -0.135 0.0024 rpy=1.5708 0 0, axis 0 0 1.0, limit effort=0.01 velocity=0.1
- added joint Untitled.099: type continuous, parent Untitled.009, child Untitled.099, origin xyz=-0.0026 0.13 0 rpy=1.5708 0 -3.14159, axis 0 0 1.0, limit effort=0.01 velocity=0.1
- added joint Untitled.100: type continuous, parent Untitled.009, child Untitled.100, origin xyz=-0.0026 -0.13 0 rpy=1.5708 0 0, axis 0 0 1.0, limit effort=0.01 velocity=0.1
- added joint Untitled.101: type fixed, parent Untitled.004, child Untitled.101, origin xyz=-0.02 0.03 -0.05 rpy=1.5708 0 0
- added joint Untitled.102: type fixed, parent Untitled.101, child Untitled.102, origin xyz=-0.01 0.05 0.03 rpy=0 0 0
- added joint Untitled.104: type fixed, parent Untitled.009, child Untitled.104, origin xyz=-0.02 0.035 -0.0524 rpy=1.5708 0 0
- added joint Untitled.105: type fixed, parent Untitled.104, child Untitled.105, origin xyz=-0.01 0.05 0.03 rpy=0 0 0
- added joint Untitled.106: type fixed, parent Untitled.004, child Untitled.106, origin xyz=0.115 -0.025 0.06 rpy=1.5708 0 -3.14159
- added joint Untitled.107: type fixed, parent Untitled.004, child Untitled.107, origin xyz=0.165 -0.025 0.06 rpy=1.5708 0 -1.5708
- added joint Untitled.108: type fixed, parent Untitled.004, child Untitled.108, origin xyz=0.17 0.025 0.06 rpy=1.5708 0 0
- added joint Untitled.109: type fixed, parent Untitled.004, child Untitled.109, origin xyz=0.11633 0.02712 0.06201 rpy=1.5708 0 1.5708
- added joint Untitled.110: type fixed, parent Untitled.052, child Untitled.110, origin xyz=-1.25101 0.00279 -0.00759 rpy=0 0 -1.5708
- added joint Untitled.111: type fixed, parent Untitled.052, child Untitled.111, origin xyz=1.24899 0.00279 0.03241 rpy=0 0 -1.5708
- joint Untitled.004: origin xyz=0 0 -1.575 rpy=0 0 0 -> xyz=0.00279 0.00101 -1.57241 rpy=0 0 0; parent Untitled.051 -> Untitled.110
- joint Untitled.009: origin xyz=0 -0.005 -1.5626 rpy=0 0 0 -> xyz=0.00279 -0.00399 -1.56 rpy=0 0 0; parent Untitled.050 -> Untitled.111
- joint Untitled.013: axis 0 0 1.0 -> (none); limit effort=0.1 velocity=1.5 -> (none); origin xyz=-0.04 0 -0.07 rpy=3.14159 0 0 -> xyz=0 0 0.055 rpy=0 0 0; parent Untitled.012 -> Untitled.053; type continuous -> fixed
- joint Untitled.039: origin xyz=-0.025 0.03 0.0476 rpy=1.5708 0 1.5708 -> xyz=-0.175 0.03 0.0476 rpy=1.5708 0 1.5708
- joint Untitled.040: origin xyz=-0.025 -0.02 0.0476 rpy=1.5708 0 -3.14159 -> xyz=-0.195 -0.02 0.0476 rpy=1.5708 0 -3.14159
- joint Untitled.045: origin xyz=0 0.005 0.1376 rpy=0 0 0 -> xyz=0.19 0.03 0.0476 rpy=1.5708 0 0
- joint Untitled.046: origin xyz=0 0 0.15 rpy=0 0 0 -> xyz=0.19 -0.02 0.0476 rpy=1.5708 0 -1.5708; parent Untitled.004 -> Untitled.009
- joint Untitled.048: origin xyz=0.10388 -0.0011 0.01673 rpy=0 0 0 -> xyz=0.10668 -8e-05 0.01932 rpy=0 0 0; parent Untitled.051 -> Untitled.110
- joint Untitled.050: origin xyz=1.25 0 -0.005 rpy=0 0 -1.5708 -> xyz=0.15 -0.02 0.0476 rpy=1.5708 0 -3.14159; parent Untitled.052 -> Untitled.009
- joint Untitled.051: origin xyz=-1.25 0 -0.005 rpy=0 0 -1.5708 -> xyz=0.14 0.03 0.0476 rpy=1.5708 0 1.5708; parent Untitled.052 -> Untitled.009
- joint Untitled.054: axis (none) -> 0 0 1.0; limit (none) -> effort=0.1 velocity=1.5; origin xyz=0 0 0.055 rpy=0 0 0 -> xyz=-0.04 0 -0.07 rpy=3.14159 0 0; parent Untitled.053 -> Untitled.012; type fixed -> continuous
- joint Untitled.055: parent Untitled.054 -> Untitled.013
- joint Untitled.057: origin xyz=0.02 0 -0.05 rpy=0 1.5708 0 -> xyz=-0.07251 -0.00274 0.02904 rpy=0 1.5708 0; parent Untitled.056 -> Untitled.110
- joint Untitled.058: parent Untitled.054 -> Untitled.013
- joint Untitled.059: origin xyz=0.0553 0.00625 0.02708 rpy=0 1.5708 0 -> xyz=0.05809 0.00726 -0.01033 rpy=0 1.5708 0; parent Untitled.050 -> Untitled.111
- joint Untitled.065: origin xyz=0.04 0 -0.05012 rpy=0 1.5708 0 -> xyz=-0.05251 0.00101 -0.01107 rpy=0 1.5708 0; parent Untitled.064 -> Untitled.111
- joint Untitled.073: origin xyz=0.025 -0.02 0.0476 rpy=1.5708 0 -1.5708 -> xyz=-0.145 -0.02 0.0476 rpy=1.5708 0 -1.5708
- joint Untitled.074: origin xyz=0.03 0.03 0.0476 rpy=1.5708 0 0 -> xyz=-0.15 0.03 0.0476 rpy=1.5708 0 0
- joint Untitled.075: origin xyz=-0.025 0.025 0.06 rpy=1.5708 0 1.5708 -> xyz=-0.195 0.025 0.06 rpy=1.5708 0 1.5708
- joint Untitled.076: origin xyz=-0.025 -0.025 0.06 rpy=1.5708 0 -3.14159 -> xyz=-0.195 -0.025 0.06 rpy=1.5708 0 -3.14159
- joint Untitled.077: origin xyz=0.025 -0.025 0.06 rpy=1.5708 0 -1.5708 -> xyz=-0.155 -0.025 0.06 rpy=1.5708 0 -1.5708
- joint Untitled.078: origin xyz=0.03 0.025 0.06 rpy=1.5708 0 0 -> xyz=-0.15 0.025 0.06 rpy=1.5708 0 0
- joint Untitled.079: origin xyz=-0.11388 1.2511 0.10827 rpy=1.5708 0 1.5708 -> xyz=-0.00145 1.25375 0.0347 rpy=3.14159 0 1.5708; parent Untitled.048 -> Untitled.013
