Commit message: aruco added

File: src/rsc/bot.urdf (robot description, URDF)
Before this commit: robot bot, 104 links, 103 joints
Links:
- added link Untitled.112, mass 0.001; visual box size=0.03 0.1 0.12
- added link Untitled.113, mass 0.001; visual box size=0.23 0.23 0.01
- added link Untitled.114, mass 0.001; visual mesh filename=Aruco.stl scale=0.0032 0.002 0.0032
- added link Untitled.115, mass 0.001; visual box size=0.04 0.07 0.005
- added link Untitled.116, mass 0.001; visual box size=0.2 0.01 0.2
- added link Untitled.117, mass 0.001; visual mesh filename=Aruco.001.stl scale=0.0028 0.002 0.0028
Joints:
- added joint Untitled.112: type fixed, parent Untitled.022, child Untitled.112, origin xyz=0.01319 0 0.13722 rpy=0 0 0
- added joint Untitled.113: type fixed, parent Untitled.112, child Untitled.113, origin xyz=-0.00319 0 0.06094 rpy=0 0 0
- added joint Untitled.114: type fixed, parent Untitled.113, child Untitled.114, origin xyz=0.05 0 0.02 rpy=1.5708 0 0
- added joint Untitled.115: type fixed, parent Untitled.035, child Untitled.115, origin xyz=0 -0.05553 0.00324 rpy=0 0 0
- added joint Untitled.116: type fixed, parent Untitled.115, child Untitled.116, origin xyz=0 -0.039 -0.00345 rpy=0 0 0
- added joint Untitled.117: type fixed, parent Untitled.116, child Untitled.117, origin xyz=0 -0.025 -0.07 rpy=0 0 0
- joint Untitled.111: origin xyz=1.24899 0.00279 0.03241 rpy=0 0 -1.5708 -> xyz=1.24899 0.00279 -0.03241 rpy=0 0 -1.5708

Commit message: full run script added

File: src/rsc/bot.urdf (robot description, URDF)
Before this commit: robot bot, 110 links, 109 joints
Links:
- added link Untitled.118, mass 0.001; visual mesh filename=12.stl scale=0.00724 0.00677 0.00094
- added link Untitled.119, mass 0.001; visual mesh filename=12.001.stl scale=0.00724 0.00677 0.00094
- link Untitled.037: geometry collision box size=0.06 0.005 0.1; visual box size=0.06 0.005 0.1
- link Untitled.038: geometry collision box size=0.06 0.005 0.1; visual box size=0.06 0.005 0.1
Joints:
- added joint Untitled.118: type fixed, parent Untitled.037, child Untitled.118, origin xyz=0 -0.02859 0.00917 rpy=-1.5708 0 0
- added joint Untitled.119: type fixed, parent Untitled.096, child Untitled.119, origin xyz=-0.00067 -0.08027 0 rpy=-1.5708 -1.5708 0
- joint Untitled.009: origin xyz=0.00279 -0.00399 -1.56 rpy=0 0 0 -> xyz=0.00279 -0.00399 -1.57241 rpy=0 0 0
- joint Untitled.111: origin xyz=1.24899 0.00279 -0.03241 rpy=0 0 -1.5708 -> xyz=1.24899 0.00279 -0.00759 rpy=0 0 -1.5708
- joint Untitled.116: origin xyz=0 -0.039 -0.00345 rpy=0 0 0 -> xyz=0 -0.039 0.10655 rpy=0 0 0
